Commit message: initial setup

File: src/my_robot/urdf/my_robot.xacro (robot description, xacro)
@@ -158,4 +158,7 @@
     </collision>
   </link>
+<!-- link for the RGB-D  -->
+  <link name="camera_link_optical">
+  </link>
 <!--joint for the left wheel-->
    <joint type="continuous" name="left_wheel_hinge">
@@ -183,5 +186,5 @@
     <axis xyz="0 1 0" rpy="0 0 0"/>
   </joint>
-<!--joint for the camera-->
+<!--joint for the LIDAR-->
    <joint type="fixed" name="hokuyo_joint">
     <origin xyz="0.15 0.0 0.1" rpy="0 0 0"/>
@@ -190,3 +193,9 @@
     <axis xyz="0 1 0" rpy="0 0 0"/>
    </joint>
+<!--joint for the RGB-D camera-->
+  <joint name="camera_optical_joint" type="fixed">
+    <origin xyz="0 0 0" rpy="-1.5707 0 -1.5707"/>
+    <parent link="camera_link"/>
+    <child link="camera_link_optical"/>
+  </joint>
 </robot>

Commit message: add/change parameters for RTAM-mapping

File: src/my_robot/urdf/my_robot.xacro (robot description, xacro)
@@ -196,5 +196,5 @@
   <joint name="camera_optical_joint" type="fixed">
     <origin xyz="0 0 0" rpy="-1.5707 0 -1.5707"/>
-    <parent link="camera_link"/>
+    <parent link="camera"/>
     <child link="camera_link_optical"/>
   </joint>
